File: HAB4-PCB1.kicad_sch (KiCad schematic)
At the start: 22 parts, among them J1 Barrel_Jack_Switch

Commit message: grounding flood plane
Parts:
- D2, D3, D4, D5: footprint LED_THT:LED_D5.0mm -> My_Footprints2:JCLPCB_THT_LED_D5.0mm
Changed lines of the file:
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@@
 			)
 		)
-		(property "Footprint" "LED_THT:LED_D5.0mm"
+		(property "Footprint" "My_Footprints2:JCLPCB_THT_LED_D5.0mm"
 			(at 93.98 130.81 0)
 			(effects
@@
 			)
 		)
-		(property "Footprint" "LED_THT:LED_D5.0mm"
+		(property "Footprint" "My_Footprints2:JCLPCB_THT_LED_D5.0mm"
 			(at 85.09 130.81 0)
 			(effects
@@
 			)
 		)
-		(property "Footprint" "LED_THT:LED_D5.0mm"
+		(property "Footprint" "My_Footprints2:JCLPCB_THT_LED_D5.0mm"
 			(at 76.2 130.81 0)
 			(effects
@@
 			)
 		)
-		(property "Footprint" "LED_THT:LED_D5.0mm"
+		(property "Footprint" "My_Footprints2:JCLPCB_THT_LED_D5.0mm"
 			(at 67.31 130.81 0)
 			(effects
